Commit message: Test lancucha ale ulozenie jest poprawne

File: szub.urdf (robot description, URDF)
Before this commit: robot sausage_hanger, 5 links, 4 joints
Links:
- removed link kielbasa_01
- removed link kielbasa_02
- removed link kielbasa_03
- removed link kielbasa_04
- removed link szubienica
- added link base_link; visual mesh filename=szubienica.gltf
- added link kielbasa_01_link; visual mesh filename=kielbasa_01.gltf
- added link kielbasa_02_link; visual mesh filename=kielbasa_02.gltf
- added link kielbasa_03_link; visual mesh filename=kielbasa_03.gltf
- added link kielbasa_04_link; visual mesh filename=kielbasa_04.gltf
- added link walec_01_link; visual mesh filename=walec_03.gltf
- added link walec_02_link; visual mesh filename=walec_02.gltf
- added link walec_03_link; visual mesh filename=walec_01.gltf
- added link walec_04_link; visual mesh filename=walec.gltf
Joints:
- added joint joint_walec_01: type fixed, parent kielbasa_01_link, child walec_01_link, origin xyz=0 0.15 0 rpy=0 0 0
- added joint joint_walec_02: type fixed, parent kielbasa_02_link, child walec_02_link, origin xyz=0 0.15 0 rpy=0 0 0
- added joint joint_walec_03: type fixed, parent kielbasa_03_link, child walec_03_link, origin xyz=0 0.15 0 rpy=0 0 0
- added joint joint_walec_04: type fixed, parent kielbasa_04_link, child walec_04_link, origin xyz=0 0.15 0 rpy=0 0 0
- joint joint_01: axis 1 0 0 -> 0 1 0; child kielbasa_01 -> kielbasa_01_link; limit lower=-1.57 upper=1.57 effort=10 velocity=1 -> lower=-1.57 upper=1.57 effort=10.0 velocity=1.0; origin xyz=0 0 -0.5 rpy=0 0 0 -> xyz=0 0 0 rpy=0 0 0; parent szubienica -> base_link
- joint joint_02: child kielbasa_02 -> kielbasa_02_link; limit lower=-1.57 upper=1.57 effort=10 velocity=1 -> lower=-1.57 upper=1.57 effort=10.0 velocity=1.0; origin xyz=0 0 -1.0 rpy=0 0 0 -> xyz=0 0.15 0 rpy=0 0 0; parent kielbasa_01 -> walec_01_link
- joint joint_03: axis 1 0 0 -> 0 1 0; child kielbasa_03 -> kielbasa_03_link; limit lower=-1.57 upper=1.57 effort=10 velocity=1 -> lower=-1.57 upper=1.57 effort=10.0 velocity=1.0; origin xyz=0 0 -1.5 rpy=0 0 0 -> xyz=0 0.15 0 rpy=0 0 0; parent kielbasa_02 -> walec_02_link
- joint joint_04: child kielbasa_04 -> kielbasa_04_link; limit lower=-1.57 upper=1.57 effort=10 velocity=1 -> lower=-1.57 upper=1.57 effort=10.0 velocity=1.0; origin xyz=0 0 -2.0 rpy=0 0 0 -> xyz=0 0.15 0 rpy=0 0 0; parent kielbasa_03 -> walec_03_link
